File: audioohmmeter.kicad_pcb (KiCad board)
At the start: 2 copper layers, 40.6 x 42.5 mm, 15 parts, among them P1 CONN_1, P2 CONN_1, SW1 SS-12F51-G6, U1 74HC04

Commit message: tweaks
Routing:
- net Net-(C1-Pad1): track 12.3 -> 10.5 mm
- net Net-(D1-Pad1): track 28.0 -> 27.5 mm
Other:
- board text added: "+"
- board text added: "-"
Changed lines of the file:
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@@
     (area 98.095199 55.829999 142.925001 107.009801)
     (thickness 1.6)
-    (drawings 10)
+    (drawings 12)
     (tracks 56)
     (zones 0)
@@
     (at 123.19 75.565 270)
     (attr smd)
-    (fp_text reference C1 (at -1.27 1.5875 270) (layer B.SilkS)
+    (fp_text reference C1 (at -0.3175 1.5875 270) (layer B.SilkS)
       (effects (font (size 1 1) (thickness 0.18)) (justify mirror))
     )
@@
       (net 2 "Net-(BT1-Pad1)"))
   )
+  (gr_text - (at 124.1425 63.1825) (layer F.SilkS)
+    (effects (font (size 3 3) (thickness 0.3)))
+  )
+  (gr_text + (at 105.0925 63.1825) (layer F.SilkS)
+    (effects (font (size 3 3) (thickness 0.3)))
+  )
   (gr_text A (at 134.9375 81.915) (layer F.SilkS)
     (effects (font (size 1.5 1.5) (thickness 0.3)))
@@
   (segment (start 107.95 75.565) (end 117.46 85.075) (width 0.3048) (layer B.Cu) (net 2))
   (segment (start 117.46 85.075) (end 121.860644 85.075) (width 0.3048) (layer B.Cu) (net 2))
+  (segment (start 117.1575 71.755) (end 118.4275 73.025) (width 0.3048) (layer B.Cu) (net 3))
+  (segment (start 121.793 73.025) (end 123.19 74.422) (width 0.3048) (layer B.Cu) (net 3))
+  (segment (start 118.4275 73.025) (end 121.793 73.025) (width 0.3048) (layer B.Cu) (net 3))
   (segment (start 123.19 74.422) (end 124.7775 72.8345) (width 0.3048) (layer B.Cu) (net 3))
   (segment (start 124.7775 72.8345) (end 124.7775 71.755) (width 0.3048) (layer B.Cu) (net 3))
-  (segment (start 124.7775 71.755) (end 123.19 70.1675) (width 0.3048) (layer F.Cu) (net 3))
-  (segment (start 118.745 70.1675) (end 117.1575 71.755) (width 0.3048) (layer F.Cu) (net 3))
-  (segment (start 123.19 70.1675) (end 118.745 70.1675) (width 0.3048) (layer F.Cu) (net 3))
   (segment (start 123.19 76.708) (end 120.904 74.422) (width 0.3048) (layer B.Cu) (net 4))
   (segment (start 120.904 74.422) (end 119.38 74.422) (width 0.3048) (layer B.Cu) (net 4))
@@
   (segment (start 117.9195 74.422) (end 119.38 74.422) (width 0.3048) (layer B.Cu) (net 4))
   (segment (start 127 76.708) (end 130.81 76.708) (width 0.3048) (layer B.Cu) (net 4))
-  (segment (start 137.4775 71.755) (end 135.5725 69.85) (width 0.3048) (layer B.Cu) (net 5))
-  (segment (start 121.601926 69.863486) (end 119.6975 71.755) (width 0.3048) (layer B.Cu) (net 5))
-  (segment (start 135.5725 69.85) (end 121.601926 69.863486) (width 0.3048) (layer B.Cu) (net 5))
+  (segment (start 119.6975 71.755) (end 120.9675 70.485) (width 0.3048) (layer F.Cu) (net 5))
+  (segment (start 136.2075 70.485) (end 137.4775 71.755) (width 0.3048) (layer F.Cu) (net 5))
+  (segment (start 120.9675 70.485) (end 136.2075 70.485) (width 0.3048) (layer F.Cu) (net 5))
   (segment (start 134.9375 79.375) (end 137.4775 76.835) (width 0.3048) (layer F.Cu) (net 5))
   (segment (start 137.4775 76.835) (end 137.4775 71.755) (width 0.3048) (layer F.Cu) (net 5))
@@
   (segment (start 125.095 73.9775) (end 127.3175 71.755) (width 0.3048) (layer F.Cu) (net 8))
   (segment (start 122.8725 73.9775) (end 125.095 73.9775) (width 0.3048) (layer F.Cu) (net 8))
-  (segment (start 120.9675 75.8825) (end 122.8725 73.9775) (width 0.3048) (layer F.Cu) (net 8))
-  (via (at 120.9675 75.8825) (size 0.86) (layers F.Cu B.Cu) (net 8))
-  (segment (start 120.142 76.708) (end 120.9675 75.8825) (width 0.3048) (layer B.Cu) (net 8))
+  (segment (start 120.65 76.2) (end 122.8725 73.9775) (width 0.3048) (layer F.Cu) (net 8))
+  (via (at 120.65 76.2) (size 0.86) (layers F.Cu B.Cu) (net 8))
+  (segment (start 120.142 76.708) (end 120.65 76.2) (width 0.3048) (layer B.Cu) (net 8))
   (segment (start 118.4275 80.645) (end 115.49 83.5825) (width 0.3048) (layer F.Cu) (net 9))
   (segment (start 115.49 83.5825) (end 115.49 94.615) (width 0.3048) (layer F.Cu) (net 9))
