File: audioohmmeter.sch (KiCad schematic (older format))
At the start: 13 parts, among them P1 CONN_1, P2 CONN_1, SW1 SS-12F51-G6, U1 74HC04

Commit message: tweaks
Other:
- note added: "+"
- note added: "-"
Changed lines of the file:
@@
 Wire Wire Line
 	9150 2450 9750 2450
+Text Notes 7550 3950 0    60   ~ 0
+-
+Text Notes 7550 4100 0    60   ~ 0
++
 $EndSCHEMATC
